File: ADC.sch (KiCad schematic (older format))
At the start: 13 parts, among them J5 TEST_1P, U11 AD1939WBSTZ, U12 74LVC1G08, U13 FOX924B - 12.288MHz

Commit message: change value of C147 capacitor and change some footprint
Parts:
- C58, C60, C61, C62, C63: footprint Capacitors_SMD:C_0603 -> Capacitors_SMD:C_0603_HandSoldering
- C59: footprint Capacitors_SMD:C_0603 -> Capacitors_SMD:C_0805_HandSoldering
Changed lines of the file:
@@
 F 0 "C58" H 2760 5270 50  0000 L CNN
 F 1 "0.1uF" H 2760 5120 50  0000 L CNN
-F 2 "Capacitors_SMD:C_0603" H 2750 5200 50  0001 C CNN
+F 2 "Capacitors_SMD:C_0603_HandSoldering" H 2750 5200 50  0001 C CNN
 F 3 "" H 2750 5200 50  0001 C CNN
 	1    2750 5200
@@
 F 0 "C59" H 3060 5270 50  0000 L CNN
 F 1 "47uF" H 3060 5120 50  0000 L CNN
-F 2 "Capacitors_SMD:C_0603" H 3050 5200 50  0001 C CNN
+F 2 "Capacitors_SMD:C_0805_HandSoldering" H 3050 5200 50  0001 C CNN
 F 3 "" H 3050 5200 50  0001 C CNN
 	1    3050 5200
@@
 F 0 "C60" H 3460 5270 50  0000 L CNN
 F 1 "0.1uF" H 3460 5120 50  0000 L CNN
-F 2 "Capacitors_SMD:C_0603" H 3450 5200 50  0001 C CNN
+F 2 "Capacitors_SMD:C_0603_HandSoldering" H 3450 5200 50  0001 C CNN
 F 3 "" H 3450 5200 50  0001 C CNN
 	1    3450 5200
@@
 F 0 "C61" H 3710 5270 50  0000 L CNN
 F 1 "10uF" H 3710 5120 50  0000 L CNN
-F 2 "Capacitors_SMD:C_0603" H 3700 5200 50  0001 C CNN
+F 2 "Capacitors_SMD:C_0603_HandSoldering" H 3700 5200 50  0001 C CNN
 F 3 "" H 3700 5200 50  0001 C CNN
 	1    3700 5200
@@
 F 0 "C62" H 4160 6120 50  0000 L CNN
 F 1 "390pF" H 4160 5970 50  0000 L CNN
-F 2 "Capacitors_SMD:C_0603" H 4150 6050 50  0001 C CNN
+F 2 "Capacitors_SMD:C_0603_HandSoldering" H 4150 6050 50  0001 C CNN
 F 3 "" H 4150 6050 50  0001 C CNN
 	1    4150 6050
@@
 F 0 "C63" H 4410 6420 50  0000 L CNN
 F 1 "5600pF" H 4410 6270 50  0000 L CNN
-F 2 "Capacitors_SMD:C_0603" H 4400 6350 50  0001 C CNN
+F 2 "Capacitors_SMD:C_0603_HandSoldering" H 4400 6350 50  0001 C CNN
 F 3 "" H 4400 6350 50  0001 C CNN
 	1    4400 6350

Commit message: fix bug and add BOM file
Parts:
- added C154, C156, C157, C158: 0.1uF, symbol C
- added C155: 0.1uf, symbol C
Connections:
- net +3.3VA: now also C156.1, C157.1, C158.1
- net +3V3: now also C154.1, C155.1
- net GNDA: now also C156.2, C157.2, C158.2
- net GNDD: now also C154.2, C155.2; no longer C58.2, C59.2, C60.2, C61.2
- new net: C58.2, C59.2, C60.2, C61.2
Changed lines of the file:
@@
 EESchema Schematic File Version 2
-LIBS:Zeabus-Elec-Hydrophone-rescue
 LIBS:power
 LIBS:device
@@
 LIBS:contrib
 LIBS:valves
+LIBS:ftdi
 LIBS:zeabus
-LIBS:ftdi
 LIBS:Zeabus-Elec-Hydrophone-cache
 EELAYER 25 0
@@
 	-1   0    0    -1
 $EndComp
-Wire Wire Line
-	7800 3100 9050 3100
 NoConn ~ 7800 3400
 NoConn ~ 7800 3700
@@
 	1    0    0    -1
 $EndComp
-Wire Wire Line
-	7800 2300 7800 2200
-Wire Wire Line
-	7800 2200 8150 2200
-Wire Wire Line
-	7800 2400 7800 2800
-Connection ~ 7800 2500
-Connection ~ 7800 2600
-Connection ~ 7800 2700
-Wire Wire Line
-	7800 2600 8150 2600
-Wire Wire Line
-	7800 3000 8500 3000
 Text HLabel 8200 3300 2    60   Input ~ 0
 SPI_CLK
@@
 Text HLabel 8200 3800 2    60   Input ~ 0
 ALRCLK
-Wire Wire Line
-	7800 3300 8200 3300
-Wire Wire Line
-	8200 3500 7800 3500
-Wire Wire Line
-	7800 3800 8200 3800
 $Comp
 L +3.3V #PWR071
@@
 	1    0    0    -1
 $EndComp
-Wire Wire Line
-	4800 1400 4800 1900
-Connection ~ 4800 1800
-Connection ~ 4800 1700
-Connection ~ 4800 1600
-Wire Wire Line
-	4800 2000 4800 2100
-Wire Wire Line
-	4800 2100 4500 2100
 Text HLabel 4500 2300 0    60   Input ~ 0
 ADC1LN
@@
 Text HLabel 4500 3000 0    60   Input ~ 0
 ADC2RP
-Wire Wire Line
-	4800 2300 4500 2300
-Wire Wire Line
-	4500 2400 4800 2400
-Wire Wire Line
-	4800 2500 4500 2500
-Wire Wire Line
-	4500 2600 4800 2600
-Wire Wire Line
-	4800 2700 4500 2700
-Wire Wire Line
-	4500 2800 4800 2800
-Wire Wire Line
-	4800 2900 4500 2900
-Wire Wire Line
-	4500 3000 4800 3000
 $Comp
 L GNDD #PWR072
@@
 	1    0    0    -1
 $EndComp
-Wire Wire Line
-	4800 3200 4800 3400
-Connection ~ 4800 3300
-Wire Wire Line
-	4500 3300 4800 3300
 Text HLabel 4500 4400 0    60   Input ~ 0
 SPI_MOSI
@@
 Text HLabel 4500 3700 0    60   Output ~ 0
 ASDATA2
-Wire Wire Line
-	4500 3600 4800 3600
-Wire Wire Line
-	4800 3700 4500 3700
-Wire Wire Line
-	4500 4400 4800 4400
-Wire Wire Line
-	4800 4500 4500 4500
 Text HLabel 2050 5600 0    60   Input ~ 0
 ~AD1939_CS
@@
 Text GLabel 2250 4100 0    60   Input ~ 0
 ~RESET
-Wire Wire Line
-	2450 4100 2250 4100
-Wire Wire Line
-	2250 3900 2450 3900
-Wire Wire Line
-	3650 4000 3650 4700
-Wire Wire Line
-	3650 4700 4800 4700
 $Comp
 L C_Small C58
@@
 	1    0    0    -1
 $EndComp
-Wire Wire Line
-	4800 4900 2750 4900
-Wire Wire Line
-	2750 4900 2750 5100
-Wire Wire Line
-	3050 5100 3050 4900
-Connection ~ 3050 4900
-Wire Wire Line
-	3450 5100 4800 5100
-Connection ~ 3700 5100
-Wire Wire Line
-	3700 5300 3700 5350
-Wire Wire Line
-	3700 5350 2750 5350
-Wire Wire Line
-	2750 5350 2750 5300
-Wire Wire Line
-	3050 5300 3050 5350
-Connection ~ 3050 5350
-Wire Wire Line
-	3450 5300 3450 5350
-Connection ~ 3450 5350
 $Comp
 L R R36
@@
 $EndComp
 $Comp
-L GNDD #PWR075
-U 1 1 59968BAE
-P 3050 5350
-F 0 "#PWR075" H 3050 5100 50  0001 C CNN
-F 1 "GNDD" H 3050 5200 50  0000 C CNN
-F 2 "" H 3050 5350 50  0001 C CNN
-F 3 "" H 3050 5350 50  0001 C CNN
-	1    3050 5350
-	1    0    0    -1
-$EndComp
-Wire Wire Line
-	2050 5600 4000 5600
-Wire Wire Line
-	4000 5600 4000 5300
-Wire Wire Line
-	4000 5300 4800 5300
-Wire Wire Line
-	2450 5400 2450 5600
-Connection ~ 2450 5600
-Wire Wire Line
-	2350 3750 2350 3900
-Connection ~ 2350 3900
-$Comp
-L +3.3V #PWR076
+L +3.3V #PWR075
 U 1 1 59968D2B
 P 2350 3450
-F 0 "#PWR076" H 2350 3300 50  0001 C CNN
+F 0 "#PWR075" H 2350 3300 50  0001 C CNN
 F 1 "+3.3V" H 2350 3590 50  0000 C CNN
 F 2 "" H 2350 3450 50  0001 C CNN
@@
 $EndComp
 $Comp
-L +3.3V #PWR077
+L +3.3V #PWR076
 U 1 1 59968D54
 P 2450 5100
-F 0 "#PWR077" H 2450 4950 50  0001 C CNN
+F 0 "#PWR076" H 2450 4950 50  0001 C CNN
 F 1 "+3.3V" H 2450 5240 50  0000 C CNN
 F 2 "" H 2450 5100 50  0001 C CNN
@@
 	0    1    1    0
 $EndComp
-Wire Wire Line
-	4300 6350 4100 6350
-Wire Wire Line
-	3800 6350 3800 6050
-Wire Wire Line
-	3800 6050 4050 6050
-Wire Wire Line
-	4250 6050 4800 6050
-Wire Wire Line
-	4800 5500 4800 6350
-Wire Wire Line
-	4800 6350 4500 6350
-Connection ~ 4800 6050
-$Comp
-L +3.3VA #PWR078
+$Comp
+L +3.3VA #PWR077
 U 1 1 599691FE
 P 3800 6050
-F 0 "#PWR078" H 3800 5900 50  0001 C CNN
+F 0 "#PWR077" H 3800 5900 50  0001 C CNN
 F 1 "+3.3VA" H 3800 6190 50  0000 C CNN
 F 2 "" H 3800 6050 50  0001 C CNN
@@
 	1    0    0    -1
 $EndComp
+Wire Wire Line
+	7800 3100 9050 3100
+Wire Wire Line
+	7800 2300 7800 2200
+Wire Wire Line
+	7800 2200 8150 2200
+Wire Wire Line
+	7800 2400 7800 2800
+Connection ~ 7800 2500
+Connection ~ 7800 2600
+Connection ~ 7800 2700
+Wire Wire Line
+	7800 2600 8150 2600
+Wire Wire Line
+	7800 3000 8500 3000
+Wire Wire Line
+	7800 3300 8200 3300
+Wire Wire Line
+	8200 3500 7800 3500
+Wire Wire Line
+	7800 3800 8200 3800
+Wire Wire Line
+	4800 2000 4800 2100
+Wire Wire Line
+	4800 2100 4500 2100
+Wire Wire Line
+	4800 2300 4500 2300
+Wire Wire Line
+	4500 2400 4800 2400
+Wire Wire Line
+	4800 2500 4500 2500
+Wire Wire Line
+	4500 2600 4800 2600
+Wire Wire Line
+	4800 2700 4500 2700
+Wire Wire Line
+	4500 2800 4800 2800
+Wire Wire Line
+	4800 2900 4500 2900
+Wire Wire Line
+	4500 3000 4800 3000
+Wire Wire Line
+	4800 3200 4800 3400
+Connection ~ 4800 3300
+Wire Wire Line
+	4500 3300 4800 3300
+Wire Wire Line
+	4500 3600 4800 3600
+Wire Wire Line
+	4800 3700 4500 3700
+Wire Wire Line
+	4500 4400 4800 4400
+Wire Wire Line
+	4800 4500 4500 4500
+Wire Wire Line
+	2450 4100 2250 4100
+Wire Wire Line
+	2250 3900 2450 3900
+Wire Wire Line
+	3650 4000 3650 4700
+Wire Wire Line
+	3650 4700 4800 4700
+Wire Wire Line
+	4800 4900 2750 4900
+Wire Wire Line
+	2750 4900 2750 5100
+Wire Wire Line
+	3050 5100 3050 4900
+Connection ~ 3050 4900
+Wire Wire Line
+	3450 5100 4800 5100
+Connection ~ 3700 5100
+Wire Wire Line
+	3700 5300 3700 5350
+Wire Wire Line
+	3700 5350 2750 5350
+Wire Wire Line
+	2750 5350 2750 5300
+Wire Wire Line
+	3050 5300 3050 5350
+Connection ~ 3050 5350
+Wire Wire Line
+	3450 5300 3450 5350
+Connection ~ 3450 5350
+Wire Wire Line
+	2050 5600 4000 5600
+Wire Wire Line
+	4000 5600 4000 5300
+Wire Wire Line
+	4000 5300 4800 5300
+Wire Wire Line
+	2450 5400 2450 5600
+Connection ~ 2450 5600
+Wire Wire Line
+	2350 3750 2350 3900
+Connection ~ 2350 3900
+Wire Wire Line
+	4300 6350 4100 6350
+Wire Wire Line
+	3800 6350 3800 6050
+Wire Wire Line
+	3800 6050 4050 6050
+Wire Wire Line
+	4250 6050 4800 6050
+Wire Wire Line
+	4800 5500 4800 6350
+Wire Wire Line
+	4800 6350 4500 6350
+Connection ~ 4800 6050
+Connection ~ 4800 1800
+Connection ~ 4800 1700
+Connection ~ 4800 1600
+Wire Wire Line
+	4800 1400 4800 1900
+$Comp
+L +3.3VA #PWR078
+U 1 1 5A72F9BE
+P 4200 1350
+F 0 "#PWR078" H 4200 1200 50  0001 C CNN
+F 1 "+3.3VA" H 4200 1490 50  0000 C CNN
+F 2 "" H 4200 1350 50  0001 C CNN
+F 3 "" H 4200 1350 50  0001 C CNN
+	1    4200 1350
+	1    0    0    -1
+$EndComp
+$Comp
+L C C157
+U 1 1 5A72FBCC
+P 4200 1600
+F 0 "C157" H 4225 1700 50  0000 L CNN
+F 1 "0.1uF" H 4225 1500 50  0000 L CNN
+F 2 "" H 4238 1450 50  0001 C CNN
+F 3 "" H 4200 1600 50  0001 C CNN
+	1    4200 1600
+	1    0    0    -1
+$EndComp
+$Comp
+L C C156
+U 1 1 5A72FC21
+P 3850 1600
+F 0 "C156" H 3875 1700 50  0000 L CNN
+F 1 "0.1uF" H 3875 1500 50  0000 L CNN
+F 2 "" H 3888 1450 50  0001 C CNN
+F 3 "" H 3850 1600 50  0001 C CNN
+	1    3850 1600
+	1    0    0    -1
+$EndComp
+$Comp
+L C C158
+U 1 1 5A72FC75
+P 4500 1600
+F 0 "C158" H 4525 1700 50  0000 L CNN
+F 1 "0.1uF" H 4525 1500 50  0000 L CNN
+F 2 "" H 4538 1450 50  0001 C CNN
+F 3 "" H 4500 1600 50  0001 C CNN
+	1    4500 1600
+	1    0    0    -1
+$EndComp
+Wire Wire Line
+	4200 1350 4200 1450
+Wire Wire Line
+	3850 1450 4500 1450
+Connection ~ 4200 1450
+Wire Wire Line
+	3850 1750 4500 1750
+Connection ~ 4200 1750
+$Comp
+L GNDA #PWR079
+U 1 1 5A72FE53
+P 4200 1800
+F 0 "#PWR079" H 4200 1550 50  0001 C CNN
+F 1 "GNDA" H 4200 1650 50  0000 C CNN
+F 2 "" H 4200 1800 50  0001 C CNN
+F 3 "" H 4200 1800 50  0001 C CNN
+	1    4200 1800
+	1    0    0    -1
+$EndComp
+$Comp
+L +3.3V #PWR080
+U 1 1 5A730005
+P 3200 1350
+F 0 "#PWR080" H 3200 1200 50  0001 C CNN
+F 1 "+3.3V" H 3200 1490 50  0000 C CNN
+F 2 "" H 3200 1350 50  0001 C CNN
+F 3 "" H 3200 1350 50  0001 C CNN
+	1    3200 1350
+	1    0    0    -1
+$EndComp
+$Comp
+L C C154
+U 1 1 5A730060
+P 3000 1550
+F 0 "C154" H 3025 1650 50  0000 L CNN
+F 1 "0.1uF" H 3025 1450 50  0000 L CNN
+F 2 "" H 3038 1400 50  0001 C CNN
+F 3 "" H 3000 1550 50  0001 C CNN
+	1    3000 1550
+	1    0    0    -1
+$EndComp
+$Comp
+L C C155
+U 1 1 5A7300B1
+P 3400 1550
+F 0 "C155" H 3425 1650 50  0000 L CNN
+F 1 "0.1uf" H 3425 1450 50  0000 L CNN
+F 2 "" H 3438 1400 50  0001 C CNN
+F 3 "" H 3400 1550 50  0001 C CNN
+	1    3400 1550
+	1    0    0    -1
+$EndComp
+Wire Wire Line
+	3000 1400 3400 1400
+Wire Wire Line
+	3200 1400 3200 1350
+Connection ~ 3200 1400
+Wire Wire Line
+	3000 1700 3400 1700
+$Comp
+L GNDD #PWR081
+U 1 1 5A730212
+P 3200 1750
+F 0 "#PWR081" H 3200 1500 50  0001 C CNN
+F 1 "GNDD" H 3200 1625 50  0000 C CNN
+F 2 "" H 3200 1750 50  0001 C CNN
+F 3 "" H 3200 1750 50  0001 C CNN
+	1    3200 1750
+	1    0    0    -1
+$EndComp
+Wire Wire Line
+	3200 1700 3200 1750
+Connection ~ 3200 1700
+Wire Wire Line
+	4200 1750 4200 1800
+$Comp
+L GNDA #PWR082
+U 1 1 5A730D12
+P 3200 5400
+F 0 "#PWR082" H 3200 5150 50  0001 C CNN
+F 1 "GNDA" H 3200 5250 50  0000 C CNN
+F 2 "" H 3200 5400 50  0001 C CNN
+F 3 "" H 3200 5400 50  0001 C CNN
+	1    3200 5400
+	1    0    0    -1
+$EndComp
+Wire Wire Line
+	3200 5350 3200 5450
+Connection ~ 3200 5350
 $EndSCHEMATC
