File: DSP-External_Port.sch (KiCad schematic (older format))
At the start: 62 parts, among them J1 JTAG, SW1 SW_DIP_x02, U1 ADSP-21489BSWZ-4B, U2 FOX924B - 25MHz

Commit message: change value of C147 capacitor and change some footprint
Parts:
- C1, C10, C11, C12, C13, C14, C15, C16, C17, C18, C19, C2, C20, C21, C22, C23, C24, C25, C26, C27, C28, C29, C3, C30, C31, C32, C33, C34, C35, C36, C37, C38, C39, C4, C40, C41, C42, C5, C6, C7, C8, C9: footprint Capacitors_SMD:C_0603 -> Capacitors_SMD:C_0603_HandSoldering
- C43, C44: footprint Capacitors_SMD:C_0603 -> Capacitors_SMD:C_0805_HandSoldering
