File: DSP-Memory.sch (KiCad schematic (older format))
At the start: 32 parts, among them J22 TEST_1P, SW2 PB, U1 ADSP-21489BSWZ-4B, U3 S29GL032N, U4 74LVC1G08, U5 74LVC1G08, U6 ADM708SARZ, Y1 CSTCC2M00G53-R0

Commit message: change value of C147 capacitor and change some footprint
Parts:
- C45, C46, C47: footprint Capacitors_SMD:C_0603 -> Capacitors_SMD:C_0603_HandSoldering
Changed lines of the file:
@@
 F 0 "C45" H 7410 4120 50  0000 L CNN
 F 1 "0.01uF" H 7410 3970 50  0000 L CNN
-F 2 "Capacitors_SMD:C_0603" H 7400 4050 50  0001 C CNN
+F 2 "Capacitors_SMD:C_0603_HandSoldering" H 7400 4050 50  0001 C CNN
 F 3 "" H 7400 4050 50  0001 C CNN
 	1    7400 4050
@@
 F 0 "C46" H 10260 3770 50  0000 L CNN
 F 1 "0.01uF" H 10260 3620 50  0000 L CNN
-F 2 "Capacitors_SMD:C_0603" H 10250 3700 50  0001 C CNN
+F 2 "Capacitors_SMD:C_0603_HandSoldering" H 10250 3700 50  0001 C CNN
 F 3 "" H 10250 3700 50  0001 C CNN
 	1    10250 3700
@@
 F 0 "C47" H 1210 7270 50  0000 L CNN
 F 1 "0.01uF" H 1210 7120 50  0000 L CNN
-F 2 "Capacitors_SMD:C_0603" H 1200 7200 50  0001 C CNN
+F 2 "Capacitors_SMD:C_0603_HandSoldering" H 1200 7200 50  0001 C CNN
 F 3 "" H 1200 7200 50  0001 C CNN
 	1    1200 7200
