File: DSP_Misc.sch (KiCad schematic (older format))
At the start: 46 parts, among them J18 TEST_1P, J2 USB_OTG, J3 TEST_1P, J4 TEST_1P, SW3 PB, SW4 PB, SW5 PB, SW6 PB, U10 FT232RQ, U7 74LVC14, U8 74AC11244, U9 NCP361SNT1G

Commit message: change value of C147 capacitor and change some footprint
Parts:
- C48, C49, C50, C51, C52, C53, C54, C55, C56, C57: footprint Capacitors_SMD:C_0603 -> Capacitors_SMD:C_0603_HandSoldering
Changed lines of the file:
@@
 F 0 "C48" H 3010 1170 50  0000 L CNN
 F 1 "0.01uF" H 3010 1020 50  0000 L CNN
-F 2 "Capacitors_SMD:C_0603" H 3000 1100 50  0001 C CNN
+F 2 "Capacitors_SMD:C_0603_HandSoldering" H 3000 1100 50  0001 C CNN
 F 3 "" H 3000 1100 50  0001 C CNN
 	1    3000 1100
@@
 F 0 "C49" H 2460 1820 50  0000 L CNN
 F 1 "1uF" H 2460 1670 50  0000 L CNN
-F 2 "Capacitors_SMD:C_0603" H 2450 1750 50  0001 C CNN
+F 2 "Capacitors_SMD:C_0603_HandSoldering" H 2450 1750 50  0001 C CNN
 F 3 "" H 2450 1750 50  0001 C CNN
 	1    2450 1750
@@
 F 0 "C50" H 2460 2970 50  0000 L CNN
 F 1 "1uF" H 2460 2820 50  0000 L CNN
-F 2 "Capacitors_SMD:C_0603" H 2450 2900 50  0001 C CNN
+F 2 "Capacitors_SMD:C_0603_HandSoldering" H 2450 2900 50  0001 C CNN
 F 3 "" H 2450 2900 50  0001 C CNN
 	1    2450 2900
@@
 F 0 "C51" H 2460 4170 50  0000 L CNN
 F 1 "1uF" H 2460 4020 50  0000 L CNN
-F 2 "Capacitors_SMD:C_0603" H 2450 4100 50  0001 C CNN
+F 2 "Capacitors_SMD:C_0603_HandSoldering" H 2450 4100 50  0001 C CNN
 F 3 "" H 2450 4100 50  0001 C CNN
 	1    2450 4100
@@
 F 0 "C52" H 2460 5370 50  0000 L CNN
 F 1 "1uF" H 2460 5220 50  0000 L CNN
-F 2 "Capacitors_SMD:C_0603" H 2450 5300 50  0001 C CNN
+F 2 "Capacitors_SMD:C_0603_HandSoldering" H 2450 5300 50  0001 C CNN
 F 3 "" H 2450 5300 50  0001 C CNN
 	1    2450 5300
@@
 F 0 "C53" H 7460 2420 50  0000 L CNN
 F 1 "0.01uF" H 7460 2270 50  0000 L CNN
-F 2 "Capacitors_SMD:C_0603" H 7450 2350 50  0001 C CNN
+F 2 "Capacitors_SMD:C_0603_HandSoldering" H 7450 2350 50  0001 C CNN
 F 3 "" H 7450 2350 50  0001 C CNN
 	1    7450 2350
@@
 F 0 "C55" H 5510 3870 50  0000 L CNN
 F 1 "0.01uF" H 5510 3720 50  0000 L CNN
-F 2 "Capacitors_SMD:C_0603" H 5500 3800 50  0001 C CNN
+F 2 "Capacitors_SMD:C_0603_HandSoldering" H 5500 3800 50  0001 C CNN
 F 3 "" H 5500 3800 50  0001 C CNN
 	1    5500 3800
@@
 F 0 "C54" H 5260 3870 50  0000 L CNN
 F 1 "1uF" H 5260 3720 50  0000 L CNN
-F 2 "Capacitors_SMD:C_0603" H 5250 3800 50  0001 C CNN
+F 2 "Capacitors_SMD:C_0603_HandSoldering" H 5250 3800 50  0001 C CNN
 F 3 "" H 5250 3800 50  0001 C CNN
 	1    5250 3800
@@
 F 0 "C57" H 7460 4420 50  0000 L CNN
 F 1 "0.1uF" H 7460 4270 50  0000 L CNN
-F 2 "Capacitors_SMD:C_0603" H 7450 4350 50  0001 C CNN
+F 2 "Capacitors_SMD:C_0603_HandSoldering" H 7450 4350 50  0001 C CNN
 F 3 "" H 7450 4350 50  0001 C CNN
 	1    7450 4350
@@
 F 0 "C56" H 7410 3870 50  0000 L CNN
 F 1 "1uF" H 7410 3720 50  0000 L CNN
-F 2 "Capacitors_SMD:C_0603" H 7400 3800 50  0001 C CNN
+F 2 "Capacitors_SMD:C_0603_HandSoldering" H 7400 3800 50  0001 C CNN
 F 3 "" H 7400 3800 50  0001 C CNN
 	1    7400 3800

Commit message: fix bug and add BOM file
Parts:
- added R101: 10k, symbol R
Connections:
- net at C54.1, C55.1, J2.1 (VBUS)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: now also R101.2
- net at J18.1, U9.4 (~FLAG): now also R101.1
Other:
- moved on the sheet: J18
