File: LNA.sch (KiCad schematic (older format))
At the start: 81 parts, among them CN1 EPS.00.250.NTN, CN2 EPS.00.250.NTN, CN3 EPS.00.250.NTN, CN4 EPS.00.250.NTN, J14 TEST_1P, J15 TEST_1P, J16 TEST_1P, J17 TEST_1P, U18 AD8334ACPZ

Commit message: change value of C147 capacitor and change some footprint
Parts:
- C112, C113, C114, C115, C116, C117, C118, C119, C120, C121, C122, C123, C124, C125, C126, C127, C128, C129, C130, C131, C132, C133, C134, C135, C136, C137, C138, C139, C140, C141, C142, C143, C144, C145, C150, C151, C152, C153: footprint Capacitors_SMD:C_0603 -> Capacitors_SMD:C_0603_HandSoldering
- CN1: footprint Zeabus:EPS-00-250 -> zeabus:EPS-00-250
