File: Zeabus-Elec-Hydrophone.sch (KiCad schematic (older format))
At the start: 5 parts, among them U21 LM1117-3.3, U22 TLV73311PDVBT, U23 LM1117-3.3

Commit message: change value of C147 capacitor and change some footprint
Parts:
- C148, C149: footprint Capacitors_SMD:C_0603 -> Capacitors_SMD:C_0603_HandSoldering
Changed lines of the file:
@@
 F 0 "C148" H 3110 1420 50  0000 L CNN
 F 1 "1uF" H 3110 1270 50  0000 L CNN
-F 2 "Capacitors_SMD:C_0603" H 3100 1350 50  0001 C CNN
+F 2 "Capacitors_SMD:C_0603_HandSoldering" H 3100 1350 50  0001 C CNN
 F 3 "" H 3100 1350 50  0001 C CNN
 	1    3100 1350
@@
 F 0 "C149" H 3060 2720 50  0000 L CNN
 F 1 "1uF" H 3060 2570 50  0000 L CNN
-F 2 "Capacitors_SMD:C_0603" H 3050 2650 50  0001 C CNN
+F 2 "Capacitors_SMD:C_0603_HandSoldering" H 3050 2650 50  0001 C CNN
 F 3 "" H 3050 2650 50  0001 C CNN
 	1    3050 2650
